File: projects/magic-wand/electronics/receiver-effects/verification/relayout-a1/receiver-effects.kicad_pcb (KiCad board)
At the start: 4 copper layers, 60 x 50 mm, 45 parts, among them J1 USB-C 5V INPUT, J2 GC9A01A 1.28in SPI, J3 4OHM BTL SPEAKER, Q1 AO3401A, U1 NINA-B302-00B-00, U2 TPS62162DSGR, U3 USBLC6-2SC6, U4 MAX98357AETE+T

Commit message: fix(magic-wand): apply receiver-effects land-pattern manufacturing corrections
- F1: Bourns MF-MSMF150/24X-2 (C78695) with datasheet land pattern
- U2: TPS62162DSGR signal pads corrected 0.60->0.50 mm per DSG0008A
- U3: add local 100nF C_BUS VBUS decoupling (C1525) with clean routing
- U4: MAX98357A TQFN pads aligned to ADI 90-0031 land pattern
- update authority metadata/extract/inventory bindings; A1 board stays DRC 0/0/0
- refresh JLCPCB bare-PCB package (new SHA-256)
Parts:
- added C_BUS: 100nF 16V X7R, MW_FACTORY:receiver-effects_C_BUS, F.Cu at (135.4, 108.0)
Routing:
- net USB_VBUS_5V: track 35.7 -> 37.9 mm
- net GND: track 1.00 -> 2.50 mm, vias 21 -> 22
