File: projects/magic-wand/electronics/receiver-effects/verification/relayout-a1/receiver-effects.kicad_sch (KiCad schematic)
At the start: 41 parts, among them J1 USB-C 5V INPUT, J2 GC9A01A 1.28in SPI, J3 4OHM BTL SPEAKER, Q1 AO3401A, U1 NINA-B302-00B-00, U2 TPS62162DSGR, U3 USBLC6-2SC6, U4 MAX98357AETE+T

Commit message: fix(magic-wand): apply receiver-effects land-pattern manufacturing corrections
- F1: Bourns MF-MSMF150/24X-2 (C78695) with datasheet land pattern
- U2: TPS62162DSGR signal pads corrected 0.60->0.50 mm per DSG0008A
- U3: add local 100nF C_BUS VBUS decoupling (C1525) with clean routing
- U4: MAX98357A TQFN pads aligned to ADI 90-0031 land pattern
- update authority metadata/extract/inventory bindings; A1 board stays DRC 0/0/0
- refresh JLCPCB bare-PCB package (new SHA-256)
Parts:
- added C_BUS: 100nF 16V X7R, MW_FACTORY:receiver-effects_C_BUS, symbol MW_FACTORY:C_BUS_0402
- F1: BOM Comments 6V resettable fuse candidate; hold/trip and enclosure-tempe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 -> 6V resettable fuse; Bourns MF-MSMF150/24X-2 (LCSC C78695); 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; LCSC C89648 -> C78695; MPN MF-MSMF150-2 -> MF-MSMF150/24X-2
Connections:
- net GND: now also C_BUS.2
- net USB_VBUS_5V: now also C_BUS.1
Other:
- moved on the sheet: C_AUDIO_10U, C_AUDIO_BULK, C_AUDIO_HF, C_BUCK_IN, C_BUCK_OUT, C_NINA_BULK, C_NINA_HF, C_USB_RAW, D1, F1, J2, J3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
